Commit message: Successfully show robot model

File: src/rt1_description/urdf/onebot_realrobot.urdf.xacro (robot description, xacro)
@@ -48,21 +48,27 @@
         <!-- 125 110 -->
     </xacro:caster>
-        <joint name="left_wheel_joint" type="fixed">
+    <!-- Remove the duplicate joint definitions and update the wheel joints to be continuous -->
+    <joint name="left_wheel_joint" type="continuous">
         <origin xyz="0.0 0.2095 0.09" rpy="0 0 0" />
         <parent link="base_link"/>
         <child link="left_wheel_link"/>
-        <axis xyz="0 0 1"/>
+        <axis xyz="0 1 0"/>  <!-- Changed to rotate around Y axis -->
     </joint>
-    <joint name="right_wheel_joint" type="fixed">
+    <joint name="right_wheel_joint" type="continuous">
         <origin xyz="0.0 -0.2095 0.09" rpy="0 0 0" />
         <parent link="base_link"/>
         <child link="right_wheel_link"/>
-        <axis xyz="0 0 1"/>
+        <axis xyz="0 1 0"/>  <!-- Changed to rotate around Y axis -->
     </joint>
+    <!-- The caster joints should probably be fixed as they are -->
     <joint name="castL_caster_base" type="fixed">
         <origin xyz="0.41966 0.12667 0.2" rpy="0 0 0" />
         <parent link="base_link"/>
         <child link="castL_caster_base"/>
-        <axis xyz="0 0 1"/>
+    </joint>
+    <joint name="castR_caster_base" type="fixed">
+        <origin xyz="0.41966 -0.12667 0.2" rpy="0 0 0" />
+        <parent link="base_link"/>
+        <child link="castR_caster_base"/>
     </joint>
     <joint name="castL_caster_link_cwheel" type="fixed">
@@ -71,10 +77,4 @@
         <child link="castL_caster_link"/>
         <axis xyz="0 1 0"/>
-    </joint>
-    <joint name="castR_caster_base" type="fixed">
-        <origin xyz="0.41966 -0.12667 0.2" rpy="0 0 0" />
-        <parent link="base_link"/>
-        <child link="castR_caster_base"/>
-        <axis xyz="0 0 1"/>
     </joint>
     <joint name="castR_caster_link_cwheel" type="fixed">

Commit message: Fix the hokuyo laser position in urdf

File: src/rt1_description/urdf/onebot_realrobot.urdf.xacro (robot description, xacro)
@@ -94,5 +94,5 @@
     </link>
     <joint name="hokuyo_joint" type="fixed">
-        <origin xyz="0.4 0 0.2" rpy="0 0 0" />
+        <origin xyz="0.4 0 0.28" rpy="0 0 0" />
         <parent link="base_link"/>
         <child link="hokuyo_link" />

Commit message: Update

File: src/rt1_description/urdf/onebot_realrobot.urdf.xacro (robot description, xacro)
@@ -98,4 +98,46 @@
         <child link="hokuyo_link" />
     </joint>
+    <!-- Add ros2_control plugin configuration -->
+    <ros2_control name="RT1Control" type="system">
+        <xacro:if value="$(arg use_sim)">
+            <!-- Simulation -->
+            <hardware>
+                <plugin>gazebo_ros2_control/GazeboSystem</plugin>
+            </hardware>
+        </xacro:if>
+        <xacro:unless value="$(arg use_sim)">
+            <!-- Real Hardware -->
+            <hardware>
+                <plugin>rt1_hardware/RT1Hardware</plugin>
+                <param name="serial_port">/dev/ttyUSB0</param>
+                <param name="baud_rate">115200</param>
+                <param name="timeout_ms">1000</param>
+            </hardware>
+        </xacro:unless>
+        <!-- Joint configurations - same for both sim and real -->
+        <joint name="left_wheel_joint">
+            <command_interface name="velocity">
+                <param name="min">-10</param>
+                <param name="max">10</param>
+            </command_interface>
+            <state_interface name="position"/>
+            <state_interface name="velocity"/>
+        </joint>
+        <joint name="right_wheel_joint">
+            <command_interface name="velocity">
+                <param name="min">-10</param>
+                <param name="max">10</param>
+            </command_interface>
+            <state_interface name="position"/>
+            <state_interface name="velocity"/>
+        </joint>
+    </ros2_control>
+    <!-- Add gazebo_ros2_control plugin -->
+    <gazebo>
+        <plugin name="gazebo_ros2_control" filename="libgazebo_ros2_control.so">
+            <parameters>$(find rt1_description)/config/controllers.yaml</parameters>
+            <robot_param_node>robot_state_publisher</robot_param_node>
+        </plugin>
+    </gazebo>
     <!--gazebo reference="hokuyo_link">
         <material>Gazebo/Blue</material>
